File: EEE3088F Micromouse Design.kicad_sch (KiCad schematic)
At the start: 79 parts, among them J1 Conn_02x16_Odd_Even, J2 Conn_01x02, J3 TYPE-C-31-M-12, Q1 AO3400A, U1 INA219AxD, U10 BQ24650, U11 DRV8833PW, U12 DRV8833PW, U2 DRV8837, U3 DRV8837, U4 DRV8837, U5 DRV8837, U6 TPS5430DDA, U7 TPS61088RHLR, U8 MCP73833-xxx-MF, U9 CH224K

Commit message: Added and fixed the external load switching to an IC instead of discrete components.
Parts:
- added C33, C34, C35, C37: 1μF, Capacitor_SMD:C_1206_3216Metric_Pad1.33x1.80mm_HandSolder, symbol Device:C_Small
- added C36, C38: 1nF, Capacitor_SMD:C_1206_3216Metric_Pad1.33x1.80mm_HandSolder, symbol Device:C_Small
- added U13: AP22966DC8-7, AP22966DC8-7:IC_AP22966DC8-7, symbol AP22966DC8-7:AP22966DC8-7
- R27, R28: value 1 -> 0.4
Connections:
- net 5V Out: now also C33.2, C34.1, U13.1_2 (VIN1), U13.4 (VBIAS), U13.6_7 (VIN2)
- net GND: now also C33.1, C34.2, C35.1, C36.2, C37.1, C38.2, U13.11 (GND), U13.15 (EXP)
- net EXT_LOAD2_OUT: now reaches J1.11 (Pin_11)
- net EXT_LOAD2_OUT: now also C37.2, U13.8_9 (VOUT2)
- net EXT_LOAD1_OUT: now reaches J1.21 (Pin_21)
- net EXT_LOAD1_OUT: now also C35.2, U13.13_14 (VOUT1)
- net CTRL_EXT_LOAD1: now reaches J1.25 (Pin_25)
- net CTRL_EXT_LOAD1: now also U13.3 (EN1)
- net CTRL_EXT_LOAD2: now reaches J1.7 (Pin_7)
- net CTRL_EXT_LOAD2: now also U13.5 (EN2)
- new net: C36.1, U13.12 (SS1)
- new net: C38.1, U13.10 (SS2)
Other:
- note added: "200mA Motor"
- note added: "500mA Motor"
- note added: "External Load Switching x2 (Downloaded Footprint Online)"
- moved on the sheet: C10, C11, C12, C13, C2, C23, C27, C28, C29, C3, C30, C31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
