File: EEE3088F Micromouse Design.kicad_pcb (KiCad board)
At the start: 2 copper layers, 70 x 78.3 mm, 98 parts, among them J1 Conn_02x16_Odd_Even, J2 Conn_01x02, J3 TYPE-C-31-M-12, Q2 AO3400A, SW1 SW_SPDT, U1 INA219AxD, U11 DRV8833PW, U12 DRV8833PW, U13 AP22966DC8-7, U14 XL1509-5.0, U15 TP4056-42-ESOP8, U2 XL1509-3.3, U3 TPS61088RHLR, U9 CH224K

Commit message: Finishing off. V2
Parts:
- removed 5VStep, CR1, CR2, CRGnd, HV, TP20, TP21, TP22, Testpoint1, vBat: TestPoint, TestPoint:TestPoint_Pad_D2.0mm
- removed C12, C13, C23, C25: 100uF, Capacitor_Tantalum_SMD:CP_EIA-3528-21_Kemet-B
- added 3v3Reg1: TestPoint, TestPoint:TestPoint_Pad_D2.0mm, F.Cu at (121.6, 81.9)
- added C53: 100uF, Capacitor_SMD:C_1206_3216Metric_Pad1.33x1.80mm_HandSolder, F.Cu at (121.8, 95.6)
- added C54: 100uF, Capacitor_SMD:C_1206_3216Metric_Pad1.33x1.80mm_HandSolder, F.Cu at (125.6, 94.0)
- added C55: 100uF, Capacitor_SMD:C_1206_3216Metric_Pad1.33x1.80mm_HandSolder, F.Cu at (118.6, 100.7)
- added C56: 100uF, Capacitor_SMD:C_1206_3216Metric_Pad1.33x1.80mm_HandSolder, F.Cu at (124.3, 101.3)
- added Comp1: TestPoint, TestPoint:TestPoint_Pad_D2.0mm, F.Cu at (101.9, 72.9)
- added HV1: TestPoint, TestPoint:TestPoint_Pad_D2.0mm, F.Cu at (110.4, 118.0)
- added VBat1: TestPoint, TestPoint:TestPoint_Pad_D2.0mm, F.Cu at (90.8, 108.2)
- added ind1: TestPoint, TestPoint:TestPoint_Pad_D2.0mm, F.Cu at (84.9, 91.9)
- added ind2: TestPoint, TestPoint:TestPoint_Pad_D2.0mm, F.Cu at (73.4, 85.3)
- C37, C38, C40, C46: footprint Capacitor_Tantalum_SMD:CP_EIA-3528-21_Kemet-B -> Capacitor_SMD:C_1206_3216Metric_Pad1.33x1.80mm_HandSolder
- moved C48 55.8 mm to (68.4, 117.0), turned to -90 degrees
- moved TP17 24.8 mm to (123.9, 86.1)
- moved C49 14.9 mm to (116.8, 105.3), turned to 0 degrees
- moved C43 7.06 mm to (114.1, 95.6)
- moved C42 7.06 mm to (118.0, 95.6)
- moved U15 0.15 mm to (87.7, 143.9)
- moved U13 0.06 mm to (101.9, 91.9)
Routing:
- net GND: track 548.2 -> 612.9 mm, vias 11 -> 13
- net /Stepped Down 5V: track 63.1 -> 101.6 mm, vias 2 -> 3
- net /HV: track 113.1 -> 136.0 mm
- net /5V Out: track 185.0 -> 202.9 mm, vias 3 -> 5
- net Net-(U3-SW_4): track 36.1 -> 50.6 mm, vias 3 -> 4
- net Net-(Q2-D): track 34.1 -> 21.0 mm, vias 2 -> 0
- net /Vcc: track 39.9 -> 49.2 mm
- net /3.3V Out: track 82.4 -> 91.1 mm
- net Net-(U2-FB): track 55.0 -> 46.8 mm
- net /CTRL_EXT_LOAD1: track 57.8 -> 64.5 mm
- net /V_Battery+: track 183.9 -> 178.3 mm, vias 6 -> 4
- net Net-(Q2-S): track 22.4 -> 18.7 mm
- net Net-(J3-CC2): track 35.1 -> 38.2 mm
- net Net-(U3-COMP): track 16.4 -> 19.1 mm
- net Net-(J3-DP1): track 26.5 -> 29.1 mm
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